File: DAQ Schematics/DAQ Schematics.sch (KiCad schematic (older format))
At the start: 5 parts

Commit message: Added code (V1.0)
Parts:
- gave numbers to parts that had none: 5
Connections:
- wire segments 77 -> 82
Other:
- note added: "Power is supplied by 5V USB connection"
- note removed: "Power is supplied by 12V barrel jack on Arduino board"
Changed lines of the file:
@@
 $EndDescr
 $Comp
-L MCU_Module:Arduino_UNO_R3 A?
+L MCU_Module:Arduino_UNO_R3 A1
 U 1 1 60FB0CEE
 P 5600 3350
-F 0 "A?" H 5600 3950 50  0000 C CNN
+F 0 "A1" H 5600 3950 50  0000 C CNN
 F 1 "Arduino_UNO_R3" H 5600 4050 50  0000 C CNN
 F 2 "Module:Arduino_UNO_R3" H 5600 3350 50  0001 C CIN
@@
 CS0
 $Comp
-L power:+5V #PWR?
+L power:+5V #PWR04
 U 1 1 60FBE811
 P 5800 2250
-F 0 "#PWR?" H 5800 2100 50  0001 C CNN
+F 0 "#PWR04" H 5800 2100 50  0001 C CNN
 F 1 "+5V" H 5815 2423 50  0000 C CNN
 F 2 "" H 5800 2250 50  0001 C CNN
@@
 $EndComp
 $Comp
-L power:+5V #PWR?
+L power:+5V #PWR05
 U 1 1 60FBF1E8
 P 8350 1050
-F 0 "#PWR?" H 8350 900 50  0001 C CNN
+F 0 "#PWR05" H 8350 900 50  0001 C CNN
 F 1 "+5V" H 8365 1223 50  0000 C CNN
 F 2 "" H 8350 1050 50  0001 C CNN
@@
 $EndComp
 $Comp
-L power:GND #PWR?
+L power:GND #PWR03
 U 1 1 60FBFACF
 P 5600 4550
-F 0 "#PWR?" H 5600 4300 50  0001 C CNN
+F 0 "#PWR03" H 5600 4300 50  0001 C CNN
 F 1 "GND" H 5605 4377 50  0000 C CNN
 F 2 "" H 5600 4550 50  0001 C CNN
@@
 	5600 4450 5600 4500
 $Comp
-L power:GND #PWR?
+L power:GND #PWR06
 U 1 1 60FC0A5E
 P 8350 1450
-F 0 "#PWR?" H 8350 1200 50  0001 C CNN
+F 0 "#PWR06" H 8350 1200 50  0001 C CNN
 F 1 "GND" H 8355 1277 50  0000 C CNN
 F 2 "" H 8350 1450 50  0001 C CNN
@@
 CS1
 $Comp
-L power:+5V #PWR?
+L power:+5V #PWR07
 U 1 1 60FC3B8D
 P 8350 1900
-F 0 "#PWR?" H 8350 1750 50  0001 C CNN
+F 0 "#PWR07" H 8350 1750 50  0001 C CNN
 F 1 "+5V" H 8365 2073 50  0000 C CNN
 F 2 "" H 8350 1900 50  0001 C CNN
@@
 $EndComp
 $Comp
-L power:GND #PWR?
+L power:GND #PWR08
 U 1 1 60FC3B93
 P 8350 2300
-F 0 "#PWR?" H 8350 2050 50  0001 C CNN
+F 0 "#PWR08" H 8350 2050 50  0001 C CNN
 F 1 "GND" H 8355 2127 50  0000 C CNN
 F 2 "" H 8350 2300 50  0001 C CNN
@@
 CS2
 $Comp
-L power:+5V #PWR?
+L power:+5V #PWR09
 U 1 1 60FC56C5
 P 8350 2750
-F 0 "#PWR?" H 8350 2600 50  0001 C CNN
+F 0 "#PWR09" H 8350 2600 50  0001 C CNN
 F 1 "+5V" H 8365 2923 50  0000 C CNN
 F 2 "" H 8350 2750 50  0001 C CNN
@@
 $EndComp
 $Comp
-L power:GND #PWR?
+L power:GND #PWR010
 U 1 1 60FC56CB
 P 8350 3150
-F 0 "#PWR?" H 8350 2900 50  0001 C CNN
+F 0 "#PWR010" H 8350 2900 50  0001 C CNN
 F 1 "GND" H 8355 2977 50  0000 C CNN
 F 2 "" H 8350 3150 50  0001 C CNN
@@
 CS3
 $Comp
-L power:+5V #PWR?
+L power:+5V #PWR011
 U 1 1 60FC61E2
 P 8350 3600
-F 0 "#PWR?" H 8350 3450 50  0001 C CNN
+F 0 "#PWR011" H 8350 3450 50  0001 C CNN
 F 1 "+5V" H 8365 3773 50  0000 C CNN
 F 2 "" H 8350 3600 50  0001 C CNN
@@
 $EndComp
 $Comp
-L power:GND #PWR?
+L power:GND #PWR012
 U 1 1 60FC61E8
 P 8350 4000
-F 0 "#PWR?" H 8350 3750 50  0001 C CNN
+F 0 "#PWR012" H 8350 3750 50  0001 C CNN
 F 1 "GND" H 8355 3827 50  0000 C CNN
 F 2 "" H 8350 4000 50  0001 C CNN
@@
 CS4
 $Comp
-L power:+5V #PWR?
+L power:+5V #PWR013
 U 1 1 60FC6F4B
 P 8350 4450
-F 0 "#PWR?" H 8350 4300 50  0001 C CNN
+F 0 "#PWR013" H 8350 4300 50  0001 C CNN
 F 1 "+5V" H 8365 4623 50  0000 C CNN
 F 2 "" H 8350 4450 50  0001 C CNN
@@
 $EndComp
 $Comp
-L power:GND #PWR?
+L power:GND #PWR014
 U 1 1 60FC6F51
 P 8350 4850
-F 0 "#PWR?" H 8350 4600 50  0001 C CNN
+F 0 "#PWR014" H 8350 4600 50  0001 C CNN
 F 1 "GND" H 8355 4677 50  0000 C CNN
 F 2 "" H 8350 4850 50  0001 C CNN
@@
 CS5
 $Comp
-L power:+5V #PWR?
+L power:+5V #PWR015
 U 1 1 60FC77D1
 P 8350 5300
-F 0 "#PWR?" H 8350 5150 50  0001 C CNN
+F 0 "#PWR015" H 8350 5150 50  0001 C CNN
 F 1 "+5V" H 8365 5473 50  0000 C CNN
 F 2 "" H 8350 5300 50  0001 C CNN
@@
 $EndComp
 $Comp
-L power:GND #PWR?
+L power:GND #PWR016
 U 1 1 60FC77D7
 P 8350 5700
-F 0 "#PWR?" H 8350 5450 50  0001 C CNN
+F 0 "#PWR016" H 8350 5450 50  0001 C CNN
 F 1 "GND" H 8355 5527 50  0000 C CNN
 F 2 "" H 8350 5700 50  0001 C CNN
@@
 Wire Wire Line
 	8350 1100 8600 1100
+Text GLabel 5000 3150 0    39   Input ~ 0
+CS0
 Text GLabel 5000 3250 0    39   Input ~ 0
-CS0
+CS1
 Text GLabel 5000 3350 0    39   Input ~ 0
-CS1
+CS2
 Text GLabel 5000 3450 0    39   Input ~ 0
-CS2
+CS3
 Text GLabel 5000 3550 0    39   Input ~ 0
-CS3
+CS4
 Text GLabel 5000 3650 0    39   Input ~ 0
-CS4
+CS5
+Text GLabel 3550 6450 0    39   Input ~ 0
+SD_CS
 Text GLabel 5000 3750 0    39   Input ~ 0
-CS5
-Text GLabel 3350 6550 0    39   Input ~ 0
 SD_CS
-Text GLabel 5000 3150 0    39   Input ~ 0
-SD_CS
-$Comp
-L Switch:SW_DIP_x01 SW?
+$Comp
+L Switch:SW_DIP_x01 SW1
 U 1 1 60FD8CD4
 P 3950 2950
-F 0 "SW?" H 3950 3217 50  0000 C CNN
+F 0 "SW1" H 3950 3217 50  0000 C CNN
 F 1 "SW_DIP_x01" H 3950 3126 50  0000 C CNN
 F 2 "" H 3950 2950 50  0001 C CNN
@@
 	5800 2250 5800 2350
 $Comp
-L power:GND #PWR?
+L power:GND #PWR01
 U 1 1 60FDE286
 P 3600 3000
-F 0 "#PWR?" H 3600 2750 50  0001 C CNN
+F 0 "#PWR01" H 3600 2750 50  0001 C CNN
 F 1 "GND" H 3605 2827 50  0000 C CNN
 F 2 "" H 3600 3000 50  0001 C CNN
@@
 	4250 2950 5100 2950
 $Comp
-L Device:LED D?
+L Device:LED D1
 U 1 1 60FE3A02
 P 4050 3450
-F 0 "D?" V 4089 3332 50  0000 R CNN
+F 0 "D1" V 4089 3332 50  0000 R CNN
 F 1 "LED" V 3998 3332 50  0000 R CNN
 F 2 "" H 4050 3450 50  0001 C CNN
@@
 $EndComp
 $Comp
-L Device:R R?
+L Device:R R1
 U 1 1 60FE4E59
 P 4400 3100
-F 0 "R?" V 4300 3100 50  0000 C CNN
+F 0 "R1" V 4300 3100 50  0000 C CNN
 F 1 "220" V 4500 3100 50  0000 C CNN
 F 2 "" V 4330 3100 50  0001 C CNN
@@
 	4050 3100 4050 3300
 $Comp
-L power:GND #PWR?
+L power:GND #PWR02
 U 1 1 60FE9B43
 P 4050 3700
-F 0 "#PWR?" H 4050 3450 50  0001 C CNN
+F 0 "#PWR02" H 4050 3450 50  0001 C CNN
 F 1 "GND" H 4055 3527 50  0000 C CNN
 F 2 "" H 4050 3700 50  0001 C CNN
@@
 SCK
 Text GLabel 5000 3950 0    39   Input ~ 0
-MOSI
+MISO
 Wire Wire Line
 	5000 3950 5100 3950
@@
 	5000 4050 5100 4050
 $Comp
-L Connector:Screw_Terminal_01x05 J?
+L Connector:Screw_Terminal_01x05 J1
 U 1 1 60FFB233
 P 10550 6000
-F 0 "J?" H 10630 6042 50  0000 L CNN
+F 0 "J1" H 10630 6042 50  0000 L CNN
 F 1 "Analog Inputs" H 10630 5951 50  0000 L CNN
 F 2 "" H 10550 6000 50  0001 C CNN
@@
 AI3
 $Comp
-L power:GND #PWR?
+L power:GND #PWR017
 U 1 1 60FFE8F5
 P 10200 6250
-F 0 "#PWR?" H 10200 6000 50  0001 C CNN
+F 0 "#PWR017" H 10200 6000 50  0001 C CNN
 F 1 "GND" H 10205 6077 50  0000 C CNN
 F 2 "" H 10200 6250 50  0001 C CNN
@@
 	6100 3650 6250 3650
 Text Notes 500  600  0    39   ~ 0
-Power is supplied by 12V barrel jack on Arduino board
+Power is supplied by 5V USB connection
+Text GLabel 5000 3850 0    39   Input ~ 0
+MOSI
+Wire Wire Line
+	5000 3850 5100 3850
+Text GLabel 3550 6750 0    39   Input ~ 0
+SCK
+Text GLabel 3550 6650 0    39   Input ~ 0
+MISO
+Text GLabel 3550 6550 0    39   Input ~ 0
+MOSI
+Wire Wire Line
+	3550 6450 3750 6450
+Wire Wire Line
+	3550 6550 3750 6550
+Wire Wire Line
+	3550 6650 3750 6650
+Wire Wire Line
+	3550 6750 3750 6750
 $EndSCHEMATC

Commit message: Updated Schematics
Parts:
- removed J1: Analog Inputs, symbol Connector:Screw_Terminal_01x05
- added J1: Analog Inputs, symbol Connector:Screw_Terminal_01x07
- added R2, R3, R4, R5, R6, R7: 10k, symbol Device:R
- D1: value LED -> RED
- SW1: value SW_DIP_x01 -> Start/Stop Logging
Connections:
- net labels added: AI4, AI5
- wire segments 82 -> 123
